File: schematic/v3/CHIP_dispv3.0.brd (EAGLE design)
At the start: 40.9 x 49.8 mm, 38 parts, among them J1 2X20-CHIPB, J3 S2B-PH-SM4-TB, Q1 NPN-DTC114YUA, Q2 PNP-DTA114YUA, U1 LMR62421, U3 DS2431P, X1 FH12-40S-0.5SH

Commit message: added v3 incl gerber
Parts:
- moved SDIO 33.9 mm to (21.6, 8.38), turned to 180 degrees
- moved Q1 5.13 mm to (33.1, 15.1), turned to 180 degrees
- moved L1 4.58 mm to (22.2, 27.1)
- moved U$2 3.97 mm to (10.4, 14.2)
- moved C7 3.45 mm to (25.7, 43.8), turned to 90 degrees
- moved X1 3.30 mm to (21.2, 5.29)
- moved C4 2.79 mm to (29.2, 31.5)
- moved C2 2.79 mm to (29.2, 33.7)
- moved C10 1.53 mm to (23.6, 43.8), turned to 90 degrees
- moved U1 1.52 mm to (28.9, 28.1)
- moved R2 1.27 mm to (28.8, 24.3), turned to 0 degrees
- moved C1 1.27 mm to (28.8, 22.1), turned to 0 degrees
- moved C3 1.27 mm to (29.2, 17.5)
- moved C5 1.27 mm to (29.2, 15.3)
- moved D1 1.27 mm to (28.1, 19.8)
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Connections:
- net GND: now also X1.23, X1.7
Routing:
- net N$1: track 45.0 -> 14.6 mm, vias 1 -> 0
- net N$27: track 42.9 -> 15.8 mm
- net PWM: track 64.2 -> 40.4 mm, vias 6 -> 3
- net N$45: track 38.1 -> 15.0 mm
- net N$25: track 39.1 -> 24.1 mm, vias 2 -> 1
- net N$44: track 36.5 -> 25.4 mm, vias 0 -> 1
- net N$28: track 33.5 -> 24.5 mm
- net N$31: track 32.3 -> 23.5 mm, vias 2 -> 0
- net N$39: track 19.0 -> 11.9 mm
- net VCC5V: track 64.7 -> 57.7 mm, vias 4 -> 2
- net LCD_D23: track 24.3 -> 17.9 mm
- net GND: track 83.9 -> 79.6 mm
- net HSYNC: track 26.0 -> 30.3 mm
- net VBAT_EXT: track 65.5 -> 61.3 mm, vias 3 -> 2
- net LCD_DE: track 27.6 -> 31.7 mm
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- added copper zone on layer 1, net FB
- added copper zone on layer 1, net VBAT_EXT
- added copper zone on layer 1, net VREG_OUTPUT

Commit message: recalc resistor to generate 19.2V
Parts:
- R2: value 140K -> 31.6k
- R3: value 11.5K -> 2.21k
Changed lines of the file:
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@@
 <attribute name="VALUE" x="35.87241875" y="27.018" size="1.27" layer="27" rot="R90"/>
 </element>
-<element name="R2" library="rcl" package="M0805" value="140K" x="28.829" y="24.3256" smashed="yes">
+<element name="R2" library="rcl" package="M0805" value="31.6k" x="28.829" y="24.3256" smashed="yes">
 <attribute name="NAME" x="25.527" y="23.0556" size="0.8128" layer="25"/>
 <attribute name="VALUE" x="27.559" y="21.7856" size="1.27" layer="27"/>
 </element>
-<element name="R3" library="rcl" package="M0805" value="11.5K" x="33.274" y="24.163" smashed="yes" rot="R90">
+<element name="R3" library="rcl" package="M0805" value="2.21k" x="33.274" y="24.163" smashed="yes" rot="R90">
 <attribute name="NAME" x="31.2674" y="24.8996" size="0.8128" layer="25" font="vector" ratio="12" rot="R270"/>
 </element>
