File: schematic/v7_ordered/CHIP_tzatziffy_v7.sch (EAGLE design)
At the start: 60 parts, among them J1 2X20-CHIP0.7_DRILL, Q2 n.a. / 2N7002ET1G, U1 n.a. / LMR62421, U3 DS2431P, X1 FH12-40S-0.5SH

Commit message: moved to ordered
Parts:
- J1: value 2X20-CHIP0.7_DRILL -> 2X20-CHIP0.8_DRILL_0.15OFFSET_LR; device JKW_CHIP:2X20-CHIP0.7_DRILL -> JKW_CHIP:2X20-CHIP0.8_DRILL_0.15OFFSET_LR
Other:
- note added: "0.7mm is actually 0.7mm and too small for the pins 0.8mm is actually 0.85mm and too lose"
Changed lines of the file:
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@@
 <part name="R13" library="rcl" deviceset="R-EU_" device="M0805" value="n.a. / 10K"/>
 <part name="U$40" library="Keyboard v0.2" deviceset="GND" device=""/>
-<part name="J1" library="JKW_CHIP" deviceset="2X20-CHIP" device="0.7_DRILL" value="2X20-CHIP0.7_DRILL"/>
+<part name="J1" library="JKW_CHIP" deviceset="2X20-CHIP" device="0.8_DRILL_0.15OFFSET_LR" value="2X20-CHIP0.8_DRILL_0.15OFFSET_LR"/>
 <part name="GND2" library="supply1" deviceset="GND" device=""/>
 <part name="SDIO" library="JKW_CHIP" deviceset="TF-HOLDER" device=""/>
@@
 Opt2) n.a.</text>
 <text x="513.08" y="241.3" size="1.778" layer="91">Opt 1) do not assemble</text>
+<text x="619.76" y="71.12" size="1.778" layer="91">0.7mm is actually 0.7mm and too small for the pins
+0.8mm is actually 0.85mm and too lose</text>
 </plain>
 <instances>
