File: schematic/v8/CHIP_tzatziffy_v8.sch (EAGLE design)
At the start: 61 parts, among them J1 2X20-CHIP0.8_DRILL_0.15OFFSET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, Q2 n.a. / 2N7002ET1G, U1 n.a. / LMR62421, U3 DS2431P, X1 FH12-40S-0.5SH

Commit message: use of new usb lib
Parts:
- removed USB: USBUSB-MICROB-SMT-DIP, Spark:USBUSB-MICROB-SMT-DIP
- added JP1: USBUSB-MICROB-SMT-DIP, JKW_CHIP:USBUSB-MICROB-SMT-DIP
- added JP2: USBMICRO_SMD, JKW_CHIP:USBMICRO_SMD
Connections:
- net GND: now also JP1.GND, JP2.GND; no longer USB.GND
- net VOUT: now also JP1.VBUS, JP2.VBUS; no longer USB.VBUS
Changed lines of the file:
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@@
 <part name="U$7" library="Keyboard v0.2" deviceset="GND" device=""/>
 <part name="Q2" library="transistor-small-signal" deviceset="BSS123" device="" value="n.a. / 2N7002ET1G"/>
-<part name="USB" library="Spark" deviceset="USB" device="USB-MICROB-SMT-DIP"/>
 <part name="U$9" library="Keyboard v0.2" deviceset="GND" device=""/>
 <part name="SJ4" library="JKW_CHIP" deviceset="SMD_SJ_3WAY_OPEN" device="T"/>
@@
 <part name="U$35" library="Keyboard v0.2" deviceset="GND" device=""/>
 <part name="R8" library="rcl" deviceset="R-EU_" device="M0805" value="10 / n.a."/>
+<part name="JP1" library="JKW_CHIP" deviceset="USB" device="USB-MICROB-SMT-DIP"/>
+<part name="JP2" library="JKW_CHIP" deviceset="USB" device="MICRO_SMD"/>
 </parts>
 <sheets>
@@
 <attribute name="VALUE" x="520.7" y="213.36" size="1.778" layer="96"/>
 </instance>
-<instance part="USB" gate="G$1" x="246.38" y="165.1" rot="MR0"/>
 <instance part="U$9" gate="M" x="254" y="160.02"/>
 <instance part="SJ4" gate="G$1" x="424.18" y="238.76" smashed="yes" rot="MR0">
@@
 <instance part="U$35" gate="M" x="548.64" y="271.78"/>
 <instance part="R8" gate="G$1" x="571.5" y="215.9" rot="R90"/>
+<instance part="JP1" gate="1" x="246.38" y="165.1" rot="MR0"/>
+<instance part="JP2" gate="1" x="271.78" y="165.1"/>
 </instances>
 <busses>
@@
 </segment>
 <segment>
-<pinref part="USB" gate="G$1" pin="GND"/>
-<wire x1="248.92" y1="165.1" x2="254" y2="165.1" width="0.1524" layer="91"/>
 <wire x1="254" y1="165.1" x2="254" y2="162.56" width="0.1524" layer="91"/>
 <pinref part="U$9" gate="M" pin="GND"/>
+<pinref part="JP1" gate="1" pin="GND"/>
+<wire x1="248.92" y1="165.1" x2="254" y2="165.1" width="0.1524" layer="91"/>
+<pinref part="JP2" gate="1" pin="GND"/>
+<wire x1="254" y1="165.1" x2="269.24" y2="165.1" width="0.1524" layer="91"/>
 </segment>
 <segment>
@@
 <net name="VOUT" class="0">
 <segment>
-<pinref part="USB" gate="G$1" pin="VBUS"/>
 <label x="264.16" y="167.64" size="1.778" layer="95" rot="MR0"/>
 <wire x1="266.7" y1="167.64" x2="266.7" y2="185.42" width="0.1524" layer="91"/>
@@
 <pinref part="J1" gate="G$1" pin="ACIN-5V"/>
 <wire x1="414.02" y1="170.18" x2="408.94" y2="170.18" width="0.1524" layer="91"/>
-<wire x1="248.92" y1="167.64" x2="266.7" y2="167.64" width="0.1524" layer="91"/>
 <wire x1="414.02" y1="185.42" x2="414.02" y2="246.38" width="0.1524" layer="91"/>
 <junction x="414.02" y="185.42"/>
@@
 <wire x1="424.18" y1="246.38" x2="414.02" y2="246.38" width="0.1524" layer="91"/>
 <label x="414.02" y="218.44" size="1.778" layer="95" rot="R90"/>
-</segment>
-<segment>
+<pinref part="JP1" gate="1" pin="VBUS"/>
+<wire x1="248.92" y1="167.64" x2="266.7" y2="167.64" width="0.1524" layer="91"/>
+<pinref part="JP2" gate="1" pin="VBUS"/>
+<wire x1="269.24" y1="167.64" x2="266.7" y2="167.64" width="0.1524" layer="91"/>
+</segment>
+<segment>

Commit message: added new smd usb
Parts:
- removed JP1: USBUSB-MICROB-SMT-DIP, JKW_CHIP:USBUSB-MICROB-SMT-DIP
- removed JP2: USBMICRO_SMD, JKW_CHIP:USBMICRO_SMD
- added J2: USB-MICROB", JKW_CHIP:USB-MICROB"
Connections:
- net GND: now also J2.GND, J2.SHIELD; no longer JP1.GND, JP2.GND
- net VOUT: now also J2.VBUS; no longer JP1.VBUS, JP2.VBUS
Other:
- note added: "CHANGELOG: _______________ v7 -> v8 - added second lowside resistor to achive 5R easier/cheaper (10||10) - changed micro USB footprint to smd"
- note removed: "CHANGELOG: _______________ v7 -> v8 added second lowside resistor to achive 5R easier/cheaper (10||10)"
Changed lines of the file:
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@@
 <?xml version="1.0" encoding="utf-8"?>
 <!DOCTYPE eagle SYSTEM "eagle.dtd">
-<eagle version="7.6.0">
+<eagle version="7.7.0">
 <drawing>
 <settings>
@@
 <part name="U$35" library="Keyboard v0.2" deviceset="GND" device=""/>
 <part name="R8" library="rcl" deviceset="R-EU_" device="M0805" value="10 / n.a."/>
-<part name="JP1" library="JKW_CHIP" deviceset="USB" device="USB-MICROB-SMT-DIP"/>
-<part name="JP2" library="JKW_CHIP" deviceset="USB" device="MICRO_SMD"/>
+<part name="J2" library="JKW_CHIP" deviceset="USB-MICROB" device="&quot;"/>
 </parts>
 <sheets>
@@
 _______________
 v7 -&gt; v8
-added second lowside resistor to achive 5R easier/cheaper (10||10)</text>
+- added second lowside resistor to achive 5R easier/cheaper (10||10)
+- changed micro USB footprint to smd</text>
 </plain>
 <instances>
@@
 <attribute name="VALUE" x="520.7" y="213.36" size="1.778" layer="96"/>
 </instance>
-<instance part="U$9" gate="M" x="254" y="160.02"/>
+<instance part="U$9" gate="M" x="248.92" y="152.4"/>
 <instance part="SJ4" gate="G$1" x="424.18" y="238.76" smashed="yes" rot="MR0">
 <attribute name="NAME" x="421.64" y="239.141" size="1.778" layer="95" rot="MR0"/>
@@
 <instance part="U$35" gate="M" x="548.64" y="271.78"/>
 <instance part="R8" gate="G$1" x="571.5" y="215.9" rot="R90"/>
-<instance part="JP1" gate="1" x="246.38" y="165.1" rot="MR0"/>
-<instance part="JP2" gate="1" x="271.78" y="165.1"/>
+<instance part="J2" gate="G$1" x="241.3" y="165.1" smashed="yes" rot="R180">
+<attribute name="NAME" x="243.84" y="154.94" size="1.778" layer="95" rot="R180"/>
+<attribute name="VALUE" x="236.22" y="172.72" size="1.778" layer="96" rot="R270"/>
+</instance>
 </instances>
 <busses>
@@
 </segment>
 <segment>
-<wire x1="254" y1="165.1" x2="254" y2="162.56" width="0.1524" layer="91"/>
+<wire x1="248.92" y1="157.48" x2="248.92" y2="154.94" width="0.1524" layer="91"/>
 <pinref part="U$9" gate="M" pin="GND"/>
-<pinref part="JP1" gate="1" pin="GND"/>
-<wire x1="248.92" y1="165.1" x2="254" y2="165.1" width="0.1524" layer="91"/>
-<pinref part="JP2" gate="1" pin="GND"/>
-<wire x1="254" y1="165.1" x2="269.24" y2="165.1" width="0.1524" layer="91"/>
+<pinref part="J2" gate="G$1" pin="GND"/>
+<wire x1="248.92" y1="157.48" x2="246.38" y2="157.48" width="0.1524" layer="91"/>
+<pinref part="J2" gate="G$1" pin="SHIELD"/>
+<wire x1="246.38" y1="170.18" x2="248.92" y2="170.18" width="0.1524" layer="91"/>
+<wire x1="248.92" y1="170.18" x2="248.92" y2="157.48" width="0.1524" layer="91"/>
+<junction x="248.92" y="157.48"/>
 </segment>
 <segment>
@@
 <wire x1="424.18" y1="246.38" x2="414.02" y2="246.38" width="0.1524" layer="91"/>
 <label x="414.02" y="218.44" size="1.778" layer="95" rot="R90"/>
-<pinref part="JP1" gate="1" pin="VBUS"/>
 <wire x1="248.92" y1="167.64" x2="266.7" y2="167.64" width="0.1524" layer="91"/>
-<pinref part="JP2" gate="1" pin="VBUS"/>
-<wire x1="269.24" y1="167.64" x2="266.7" y2="167.64" width="0.1524" layer="91"/>
-</segment>
-<segment>
+<pinref part="J2" gate="G$1" pin="VBUS"/>
+<wire x1="246.38" y1="167.64" x2="266.7" y2="167.64" width="0.1524" layer="91"/>
+<junction x="266.7" y="167.64"/>
+</segment>
+<segment>
