File: schematic/v8_ordered/CHIP_tzatziffy_v8.sch (EAGLE design)
At the start: 61 parts, among them J1 2X20-CHIP0.8_DRILL_0.15OFFSET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, J2 USB-MICROB", Q2 n.a. / 2N7002ET1G, U1 n.a. / LMR62421, U3 DS2431P, X1 FH12-40S-0.5SH

Commit message: changed chip footprint to clamp via row claming 0.1mm outside and ordered v8
Parts:
- removed J2: USB-MICROB", JKW_CHIP:USB-MICROB"
- removed U3: DS2431P, Keyboard v0_5:DS2431P
- added JP1: USBMICRO_SMD, JKW_CHIP:USBMICRO_SMD
- added U2: DS2431P, JKW_CHIP:DS2431P
- J1: value 2X20-CHIP0.8_DRILL_0.15OFFSET_LR -> 2X20-CHIP0.9DRILLS_2; device JKW_CHIP:2X20-CHIP0.8_DRILL_0.15OFFSET_LR -> JKW_CHIP:2X20-CHIP0.9DRILLS_2
Connections:
- net 1WIRE: now also U2.IO; no longer U3.IO
- net GND: now also JP1.GND, U2.GND; no longer J2.GND, J2.SHIELD, U3.GND
- net VOUT: now also JP1.VBUS; no longer J2.VBUS
Other:
- note added: "CHANGELOG: _______________ v7 -> v8 - added second lowside resistor to achive 5R easier/cheaper (10||10) - changed micro USB footprint to smd - changed drills from 0.8mm to 0.9mm and 0.1mm offset per bank - increased DS2431 footprint"
- note removed: "CHANGELOG: _______________ v7 -> v8 - added second lowside resistor to achive 5R easier/cheaper (10||10) - changed micro USB footprint to smd"
Changed lines of the file:
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@@
 <?xml version="1.0" encoding="utf-8"?>
 <!DOCTYPE eagle SYSTEM "eagle.dtd">
-<eagle version="7.7.0">
+<eagle version="7.6.0">
 <drawing>
 <settings>
@@
 <part name="R12" library="rcl" deviceset="R-EU_" device="M0805" value="4.7K"/>
 <part name="SUPPLY13" library="Keyboard v0.3" deviceset="VCC3V3" device=""/>
-<part name="U3" library="Keyboard v0_5" deviceset="DS2431" device="P"/>
 <part name="D1" library="Keyboard v0_5" deviceset="DIODE_SCHTKY_B240" device="" value="B240A"/>
 <part name="R13" library="rcl" deviceset="R-EU_" device="M0805" value="n.a. / 10K"/>
 <part name="U$40" library="Keyboard v0.2" deviceset="GND" device=""/>
-<part name="J1" library="JKW_CHIP" deviceset="2X20-CHIP" device="0.8_DRILL_0.15OFFSET_LR" value="2X20-CHIP0.8_DRILL_0.15OFFSET_LR"/>
+<part name="J1" library="JKW_CHIP" deviceset="2X20-CHIP" device="0.9DRILLS_2" value="2X20-CHIP0.9DRILLS_2"/>
 <part name="GND2" library="supply1" deviceset="GND" device=""/>
 <part name="SDIO" library="JKW_CHIP" deviceset="TF-HOLDER" device=""/>
@@
 <part name="U$35" library="Keyboard v0.2" deviceset="GND" device=""/>
 <part name="R8" library="rcl" deviceset="R-EU_" device="M0805" value="10 / n.a."/>
-<part name="J2" library="JKW_CHIP" deviceset="USB-MICROB" device="&quot;"/>
+<part name="JP1" library="JKW_CHIP" deviceset="USB" device="MICRO_SMD"/>
+<part name="U2" library="JKW_CHIP" deviceset="DS2431" device="P"/>
 </parts>
 <sheets>
@@
 v7 -&gt; v8
 - added second lowside resistor to achive 5R easier/cheaper (10||10)
-- changed micro USB footprint to smd</text>
+- changed micro USB footprint to smd
+- changed drills from 0.8mm to 0.9mm and 0.1mm offset per bank
+- increased DS2431 footprint</text>
 </plain>
 <instances>
@@
 <instance part="R12" gate="G$1" x="261.62" y="83.82" rot="R90"/>
 <instance part="SUPPLY13" gate="+5V" x="261.62" y="93.98"/>
-<instance part="U3" gate="G$1" x="246.38" y="73.66"/>
 <instance part="D1" gate="G$1" x="535.94" y="261.62"/>
 <instance part="R13" gate="G$1" x="508" y="220.98" rot="R90"/>
@@
 <attribute name="VALUE" x="520.7" y="213.36" size="1.778" layer="96"/>
 </instance>
-<instance part="U$9" gate="M" x="248.92" y="152.4"/>
+<instance part="U$9" gate="M" x="266.7" y="154.94"/>
 <instance part="SJ4" gate="G$1" x="424.18" y="238.76" smashed="yes" rot="MR0">
 <attribute name="NAME" x="421.64" y="239.141" size="1.778" layer="95" rot="MR0"/>
@@
 <instance part="U$35" gate="M" x="548.64" y="271.78"/>
 <instance part="R8" gate="G$1" x="571.5" y="215.9" rot="R90"/>
-<instance part="J2" gate="G$1" x="241.3" y="165.1" smashed="yes" rot="R180">
-<attribute name="NAME" x="243.84" y="154.94" size="1.778" layer="95" rot="R180"/>
-<attribute name="VALUE" x="236.22" y="172.72" size="1.778" layer="96" rot="R270"/>
-</instance>
+<instance part="JP1" gate="1" x="251.46" y="162.56" rot="MR0"/>
+<instance part="U2" gate="G$1" x="246.38" y="73.66"/>
 </instances>
 <busses>
@@
 <pinref part="U$36" gate="M" pin="GND"/>
 <wire x1="243.84" y1="60.96" x2="243.84" y2="55.88" width="0.1524" layer="91"/>
-<pinref part="U3" gate="G$1" pin="GND"/>
+<pinref part="U2" gate="G$1" pin="GND"/>
 </segment>
 <segment>
@@
 </segment>
 <segment>
-<wire x1="248.92" y1="157.48" x2="248.92" y2="154.94" width="0.1524" layer="91"/>
 <pinref part="U$9" gate="M" pin="GND"/>
-<pinref part="J2" gate="G$1" pin="GND"/>
-<wire x1="248.92" y1="157.48" x2="246.38" y2="157.48" width="0.1524" layer="91"/>
-<pinref part="J2" gate="G$1" pin="SHIELD"/>
-<wire x1="246.38" y1="170.18" x2="248.92" y2="170.18" width="0.1524" layer="91"/>
-<wire x1="248.92" y1="170.18" x2="248.92" y2="157.48" width="0.1524" layer="91"/>
-<junction x="248.92" y="157.48"/>
+<wire x1="254" y1="162.56" x2="266.7" y2="162.56" width="0.1524" layer="91"/>
+<wire x1="266.7" y1="162.56" x2="266.7" y2="157.48" width="0.1524" layer="91"/>
+<pinref part="JP1" gate="1" pin="GND"/>
 </segment>
 <segment>
@@
 </segment>
 <segment>
-<wire x1="256.54" y1="76.2" x2="261.62" y2="76.2" width="0.1524" layer="91"/>
 <wire x1="261.62" y1="76.2" x2="261.62" y2="78.74" width="0.1524" layer="91"/>
 <pinref part="R12" gate="G$1" pin="1"/>
 <wire x1="261.62" y1="76.2" x2="271.78" y2="76.2" width="0.1524" layer="91"/>
 <junction x="261.62" y="76.2"/>
-<pinref part="U3" gate="G$1" pin="IO"/>
 <label x="264.16" y="76.2" size="1.778" layer="95" font="vector" ratio="12"/>
+<pinref part="U2" gate="G$1" pin="IO"/>
+<wire x1="256.54" y1="76.2" x2="261.62" y2="76.2" width="0.1524" layer="91"/>
 </segment>
 </net>
@@
 <net name="VOUT" class="0">
 <segment>
-<label x="264.16" y="167.64" size="1.778" layer="95" rot="MR0"/>
-<wire x1="266.7" y1="167.64" x2="266.7" y2="185.42" width="0.1524" layer="91"/>
+<label x="266.7" y="175.26" size="1.778" layer="95" rot="MR270"/>
+<wire x1="266.7" y1="165.1" x2="266.7" y2="185.42" width="0.1524" layer="91"/>
 <wire x1="266.7" y1="185.42" x2="414.02" y2="185.42" width="0.1524" layer="91"/>
 <wire x1="414.02" y1="185.42" x2="414.02" y2="170.18" width="0.1524" layer="91"/>
@@
 <wire x1="424.18" y1="246.38" x2="414.02" y2="246.38" width="0.1524" layer="91"/>
 <label x="414.02" y="218.44" size="1.778" layer="95" rot="R90"/>
-<wire x1="248.92" y1="167.64" x2="266.7" y2="167.64" width="0.1524" layer="91"/>
-<pinref part="J2" gate="G$1" pin="VBUS"/>
-<wire x1="246.38" y1="167.64" x2="266.7" y2="167.64" width="0.1524" layer="91"/>
-<junction x="266.7" y="167.64"/>
-</segment>
-<segment>
+<wire x1="254" y1="165.1" x2="266.7" y2="165.1" width="0.1524" layer="91"/>
+<pinref part="JP1" gate="1" pin="VBUS"/>
+</segment>
+<segment>

Commit message: added and gate
Parts:
- added IC1: 74AHC1G08DCK, 74xx-little-us:74AHC1G08DCK
Connections:
- net EN: now also IC1A.I0
- net GND: now also IC1P.GND
- net PWM: now also IC1A.I1, IC1A.O
- net VCC3V3: now also IC1P.VCC
Other:
- moved on the sheet: SJ1
Changed lines of the file:
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@@
 <?xml version="1.0" encoding="utf-8"?>
 <!DOCTYPE eagle SYSTEM "eagle.dtd">
-<eagle version="7.6.0">
+<eagle version="7.7.0">
 <drawing>
 <settings>
@@
 <part name="JP1" library="JKW_CHIP" deviceset="USB" device="MICRO_SMD"/>
 <part name="U2" library="JKW_CHIP" deviceset="DS2431" device="P"/>
+<part name="IC1" library="74xx-little-us" deviceset="74*1G08" device="DCK" technology="AHC"/>
+<part name="U$37" library="Keyboard v0.2" deviceset="GND" device=""/>
+<part name="SUPPLY5" library="Keyboard v0.3" deviceset="VCC3V3" device=""/>
 </parts>
 <sheets>
@@
 <wire x1="233.68" y1="213.36" x2="233.68" y2="109.22" width="0.4064" layer="94" style="shortdash"/>
 <wire x1="284.48" y1="213.36" x2="284.48" y2="109.22" width="0.4064" layer="94" style="shortdash"/>
-<wire x1="406.4" y1="294.64" x2="233.68" y2="294.64" width="0.4064" layer="94" style="shortdash"/>
-<wire x1="406.4" y1="228.6" x2="233.68" y2="228.6" width="0.4064" layer="94" style="shortdash"/>
+<wire x1="398.78" y1="294.64" x2="233.68" y2="294.64" width="0.4064" layer="94" style="shortdash"/>
+<wire x1="398.78" y1="228.6" x2="233.68" y2="228.6" width="0.4064" layer="94" style="shortdash"/>
 <wire x1="233.68" y1="294.64" x2="233.68" y2="228.6" width="0.4064" layer="94" style="shortdash"/>
-<wire x1="406.4" y1="294.64" x2="406.4" y2="228.6" width="0.4064" layer="94" style="shortdash"/>
+<wire x1="398.78" y1="294.64" x2="398.78" y2="228.6" width="0.4064" layer="94" style="shortdash"/>
 <text x="236.22" y="292.1" size="1.778" layer="94">Audio</text>
-<wire x1="408.94" y1="294.64" x2="599.44" y2="294.64" width="0.4064" layer="94" style="shortdash"/>
+<wire x1="401.32" y1="294.64" x2="599.44" y2="294.64" width="0.4064" layer="94" style="shortdash"/>
 <wire x1="490.22" y1="200.66" x2="599.44" y2="200.66" width="0.4064" layer="94" style="shortdash"/>
 <wire x1="490.22" y1="200.66" x2="490.22" y2="215.9" width="0.4064" layer="94" style="shortdash"/>
-<wire x1="490.22" y1="215.9" x2="408.94" y2="215.9" width="0.4064" layer="94" style="shortdash"/>
-<wire x1="408.94" y1="215.9" x2="408.94" y2="294.64" width="0.4064" layer="94" style="shortdash"/>
+<wire x1="490.22" y1="215.9" x2="401.32" y2="215.9" width="0.4064" layer="94" style="shortdash"/>
+<wire x1="401.32" y1="215.9" x2="401.32" y2="294.64" width="0.4064" layer="94" style="shortdash"/>
 <wire x1="599.44" y1="200.66" x2="599.44" y2="294.64" width="0.4064" layer="94" style="shortdash"/>
-<text x="411.48" y="292.1" size="1.778" layer="94">DC/DC converter</text>
+<text x="403.86" y="292.1" size="1.778" layer="94">DC/DC converter</text>
 <text x="579.12" y="210.82" size="1.778" layer="91">0.2V
 @40mA
@@
 - changed drills from 0.8mm to 0.9mm and 0.1mm offset per bank
 - increased DS2431 footprint</text>
+<text x="427.99" y="251.968" size="1.778" layer="99">&lt;- cut here</text>
 </plain>
 <instances>
@@
 <instance part="GND1" gate="1" x="480.06" y="157.48"/>
 <instance part="U$2" gate="G$1" x="279.4" y="48.26"/>
-<instance part="SJ1" gate="G$1" x="447.04" y="238.76"/>
-<instance part="SUPPLY2" gate="+5V" x="447.04" y="251.46"/>
+<instance part="SJ1" gate="G$1" x="449.58" y="238.76" smashed="yes">
+<attribute name="NAME" x="452.12" y="239.141" size="1.778" layer="95"/>
+</instance>
+<instance part="SUPPLY2" gate="+5V" x="449.58" y="251.46"/>
 <instance part="L2" gate="G$1" x="500.38" y="276.86" smashed="yes">
 <attribute name="NAME" x="495.0206" y="273.2786" size="2.0828" layer="95" ratio="10" rot="SR0"/>
@@
 <instance part="JP1" gate="1" x="251.46" y="162.56" rot="MR0"/>
 <instance part="U2" gate="G$1" x="246.38" y="73.66"/>
+<instance part="IC1" gate="A" x="419.1" y="264.16" rot="R90"/>
+<instance part="IC1" gate="P" x="406.4" y="269.24" smashed="yes">
+<attribute name="NAME" x="403.225" y="272.415" size="1.778" layer="95" rot="R270"/>
+</instance>
+<instance part="U$37" gate="M" x="406.4" y="254"/>
+<instance part="SUPPLY5" gate="+5V" x="406.4" y="284.48"/>
 </instances>
 <busses>
@@
 <pinref part="U$35" gate="M" pin="GND"/>
 <wire x1="548.64" y1="274.32" x2="548.64" y2="276.86" width="0.1524" layer="91"/>
+</segment>
+<segment>
+<pinref part="IC1" gate="P" pin="GND"/>
+<pinref part="U$37" gate="M" pin="GND"/>
+<wire x1="406.4" y1="261.62" x2="406.4" y2="256.54" width="0.1524" layer="91"/>
 </segment>
 </net>
@@
 <wire x1="414.02" y1="81.28" x2="414.02" y2="93.98" width="0.1524" layer="91"/>
 </segment>
+<segment>
+<pinref part="SUPPLY5" gate="+5V" pin="VCC3V3"/>
+<pinref part="IC1" gate="P" pin="VCC"/>
+<wire x1="406.4" y1="276.86" x2="406.4" y2="281.94" width="0.1524" layer="91"/>
+</segment>
 </net>
 <net name="LCD_D5" class="0">
@@
 <pinref part="SUPPLY2" gate="+5V" pin="VCC5V"/>
 <pinref part="SJ1" gate="G$1" pin="1"/>
-<wire x1="447.04" y1="243.84" x2="447.04" y2="248.92" width="0.1524" layer="91"/>
+<wire x1="449.58" y1="243.84" x2="449.58" y2="248.92" width="0.1524" layer="91"/>
 </segment>
 </net>
@@
 <label x="411.48" y="162.56" size="1.778" layer="95" font="vector" ratio="12"/>
 <wire x1="419.1" y1="193.04" x2="419.1" y2="213.36" width="0.1524" layer="91"/>
-<wire x1="447.04" y1="213.36" x2="419.1" y2="213.36" width="0.1524" layer="91"/>
+<wire x1="449.58" y1="213.36" x2="419.1" y2="213.36" width="0.1524" layer="91"/>
 <pinref part="J1" gate="G$1" pin="VBAT-EXT"/>
 <pinref part="SJ1" gate="G$1" pin="3"/>
 <wire x1="266.7" y1="200.66" x2="243.84" y2="200.66" width="0.1524" layer="91"/>
-<wire x1="447.04" y1="213.36" x2="447.04" y2="233.68" width="0.1524" layer="91"/>
+<wire x1="449.58" y1="213.36" x2="449.58" y2="233.68" width="0.1524" layer="91"/>
 <pinref part="BV" gate="P" pin="P"/>
-<label x="447.04" y="218.44" size="1.778" layer="95" rot="R90"/>
+<label x="449.58" y="218.44" size="1.778" layer="95" rot="R90"/>
 <wire x1="266.7" y1="200.66" x2="266.7" y2="193.04" width="0.1524" layer="91"/>
 <wire x1="266.7" y1="193.04" x2="419.1" y2="193.04" width="0.1524" layer="91"/>
@@
 <wire x1="487.68" y1="254" x2="485.14" y2="254" width="0.1524" layer="91"/>
 <label x="477.52" y="220.98" size="1.778" layer="95" rot="R90"/>
-<wire x1="325.12" y1="195.58" x2="477.52" y2="195.58" width="0.1524" layer="91"/>
+<wire x1="325.12" y1="195.58" x2="416.56" y2="195.58" width="0.1524" layer="91"/>
+<wire x1="416.56" y1="195.58" x2="477.52" y2="195.58" width="0.1524" layer="91"/>
 <wire x1="477.52" y1="195.58" x2="477.52" y2="254" width="0.1524" layer="91"/>
 <wire x1="487.68" y1="254" x2="477.52" y2="254" width="0.1524" layer="91"/>
@@
 <junction x="487.68" y="254"/>
 <wire x1="487.68" y1="254" x2="492.76" y2="254" width="0.1524" layer="91"/>
+<pinref part="IC1" gate="A" pin="I0"/>
+<wire x1="416.56" y1="251.46" x2="416.56" y2="195.58" width="0.1524" layer="91"/>
+<junction x="416.56" y="195.58"/>
 </segment>
 <segment>
@@
 <pinref part="C2" gate="G$1" pin="1"/>
 <pinref part="SJ1" gate="G$1" pin="2"/>
-<wire x1="439.42" y1="238.76" x2="441.96" y2="238.76" width="0.1524" layer="91"/>
+<wire x1="441.96" y1="238.76" x2="444.5" y2="238.76" width="0.1524" layer="91"/>
 <pinref part="SJ4" gate="G$1" pin="2"/>
-<wire x1="429.26" y1="238.76" x2="439.42" y2="238.76" width="0.1524" layer="91"/>
-<junction x="439.42" y="238.76"/>
-<wire x1="439.42" y1="261.62" x2="439.42" y2="238.76" width="0.1524" layer="91"/>
-<wire x1="459.74" y1="261.62" x2="439.42" y2="261.62" width="0.1524" layer="91"/>
+<wire x1="429.26" y1="238.76" x2="441.96" y2="238.76" width="0.1524" layer="91"/>
+<junction x="441.96" y="238.76"/>
+<wire x1="441.96" y1="261.62" x2="441.96" y2="238.76" width="0.1524" layer="91"/>
+<wire x1="459.74" y1="261.62" x2="441.96" y2="261.62" width="0.1524" layer="91"/>
 <pinref part="C4" gate="G$1" pin="1"/>
 <wire x1="459.74" y1="254" x2="459.74" y2="261.62" width="0.1524" layer="91"/>
@@
 <label x="469.9" y="262.89" size="1.778" layer="95"/>
 <pinref part="U$27" gate="G$1" pin="IN"/>
-<wire x1="447.04" y1="287.02" x2="439.42" y2="287.02" width="0.1524" layer="91"/>
-<wire x1="439.42" y1="287.02" x2="439.42" y2="261.62" width="0.1524" layer="91"/>
-<junction x="439.42" y="261.62"/>
+<wire x1="447.04" y1="287.02" x2="441.96" y2="287.02" width="0.1524" layer="91"/>
+<wire x1="441.96" y1="287.02" x2="441.96" y2="261.62" width="0.1524" layer="91"/>
+<junction x="441.96" y="261.62"/>
 </segment>
 </net>
@@
 <net name="PWM" class="0">
 <segment>
-<pinref part="U$27" gate="G$1" pin="CTRL"/>
 <wire x1="408.94" y1="149.86" x2="421.64" y2="149.86" width="0.1524" layer="91"/>
 <label x="411.48" y="149.86" size="1.778" layer="95" font="vector" ratio="12"/>
@@
 <junction x="508" y="231.14"/>
 <label x="421.64" y="218.44" size="1.778" layer="95" rot="R90"/>
-<wire x1="447.04" y1="276.86" x2="421.64" y2="276.86" width="0.1524" layer="91"/>
-<wire x1="421.64" y1="276.86" x2="421.64" y2="231.14" width="0.1524" layer="91"/>
 <junction x="421.64" y="231.14"/>
-</segment>
-</net>
+<pinref part="IC1" gate="A" pin="I1"/>
+<wire x1="421.64" y1="251.46" x2="421.64" y2="248.92" width="0.1524" layer="91"/>
+<wire x1="421.64" y1="248.92" x2="421.64" y2="231.14" width="0.1524" layer="91"/>
+<wire x1="421.64" y1="248.92" x2="426.72" y2="248.92" width="0.1524" layer="91"/>
+<pinref part="U$27" gate="G$1" pin="CTRL"/>
+<wire x1="447.04" y1="276.86" x2="426.72" y2="276.86" width="0.1524" layer="91"/>
+<pinref part="IC1" gate="A" pin="O"/>
+<wire x1="426.72" y1="276.86" x2="419.1" y2="276.86" width="0.1524" layer="91"/>
+<wire x1="426.72" y1="248.92" x2="426.72" y2="276.86" width="0.1524" layer="91"/>
+<junction x="421.64" y="248.92"/>
+<junction x="426.72" y="276.86"/>
+</segment>
+</net>
